File: Micropendous/Design/Micropendous2/Micropendous2.sch (KiCad schematic (older format))
At the start: 75 parts, among them IC1 ATMEGA32U4, IC2 ST1L05B, K1 Vcc_Sel, SW1 RESET, SW2 HWB, U1 Micropendous2, U3 USBCONN, U4 CONN_MICROSD, X1 8MHz

Commit message: Complete renaming.
Parts:
- added C26: 4.7uF, symbol C_MINI
- added C27: 0.1uF, symbol C_MINI
- added V76, V77, V78, V79, V80, V81, V82, V83, V84: VIA, symbol VIA
- R5, R8: value 47k -> 43k
- U4: value CONN_MICROSD -> microSD
Connections:
- net labels added: 3.56V
- net labels removed: 3.65V
- wire segments 114 -> 127
- no-connect marks 4 -> 5
Other:
- moved on the sheet: V43, V45
