File: Micropendous/Design/Micropendous-32U4/Micropendous-32U4.sch (KiCad schematic (older format))
At the start: 36 parts, among them IC1 ATMEGA32U4-AU, K1 Vcc_Sel, SW1 RESET, SW2 HWB, U1 Micropendous-32U4, U3 USB-miniB, U4 CONN_MICROSD, U5 1117-Adj, X1 8MHz

Commit message: Updated Micropendous-32U4 with new microSD connector.
Parts:
- added V10, V23, V31, V32, V33, V34, V35, V38, V40, V41, V42, V43, V45, V46, V47, V48, V49, V51, V56, V57, V58, V59, V60, V61, V62, V65, V66, V70, V73, V74, V75, V76, V77, V79, V80, V81, V82, V83, V85, V86, V87, V88, V89, V90, V91: VIA, symbol VIA
- C24: value 22uF -> 10uF
- U4: value CONN_MICROSD -> microSD
Connections:
- net labels added: REG_GND
- wire segments 87 -> 126
Other:
- note added: "AVR will only run reliably at 3.3V Vcc if using 8MHz crystal"
- note added: "Amphenol 101-00303-68-1"
- note added: "Vias"
- note removed: "3M 290805"
- note removed: "AVR will only run at 3.3V Vcc if clock is 8MHz"
- note removed: "Digi-Key 3M5607CT-ND"
