File: Micropendous/Design/Micropendous/Micropendous.sch (KiCad schematic (older format))
At the start: 266 parts, among them IC1 AT90USB1287, IC2 1117-5V, IC3 ISL54200IRZ, IC4 74VHC573, IC5 CY7C1019D_5V_1MBIT_SRAM, IC6 TXS0108, IC7 1117-3.3V, J2 DC_POWER_JACK, P1 USB_B/^A, P2 ADC, P3 Power, P4 GPIO1, P5 GPIO2, P6 GPIO3, P7 VT, Q1 MOSFET_P_OPENDOUS, SW1 RESET, SW2 HWB, U1 USB-B, U2 USB-A, U3 CONN_MMC-SD, U4 JTAG, U7 USB-miniB, X1 16MHz

Commit message: Updated Micropendous and Micropendous-DIP AT90USB1287-based designs.
Parts:
- removed C15, C19, C33: 10uF, symbol C_MINI
- removed C16, C22, C29, C30, C31, C32, C34, C38, C40: 0.1uF, symbol C_MINI
- removed CR1, CR2, CR3: ESD_ZENER, symbol ESD_ZENER
- removed D3: MBRX120, symbol D_RECTIFIER
- removed IC2: 1117-5V, symbol TLV1117
- removed IC3: ISL54200IRZ, symbol ISL54200IRZ
- removed IC6: TXS0108, symbol TXB0108
- removed IC7: 1117-3.3V, symbol TLV1117
- removed J2: DC_POWER_JACK, symbol DC_POWER_JACK
- removed P1: USB_B/^A, symbol CONN_2
- removed P2: ADC, symbol CONN_8
- removed P3: Power, symbol CONN_8
- removed P4: GPIO1, symbol CONN_8X2
- removed P5: GPIO2, symbol CONN_8X2
- removed P6: GPIO3, symbol CONN_10X2_OPENDOUS
- removed P7: VT, symbol CONN_2
- removed R1, R2, R3, R4, R5: 22, symbol R_MINI
- removed R10: 15k, symbol R_MINI
- removed R15: 0, symbol R_MINI
- removed R16: 47k, symbol R_MINI
- removed U1: USB-B, symbol USBCONN-HOSTCAPABLE
- removed U3: CONN_MMC-SD, symbol CONN_SD
- removed U7: USB-miniB, symbol USBCONN-HOSTCAPABLE
- removed V1, V10, V100, V101, V102, V103, V104, V105, V106, V107, V108, V109, V11, V110, V111, V112, V113, V114, V115, V116, V117, V118, V119, V12, V120, V121, V122, V123, V124, V125, V126, V127, V128, V129, V13, V130, V131, V132, V133, V134, V135, V136, V137, V138, V139, V14, V140, V141, V142, V143, V144, V145, V146, V147, V148, V149, V15, V150, V151, V152, V153, V154, V155, V156, V157, V158, V159, V16, V160, V161, V162, V163, V164, V165, V166, V167, V168, V169, V17, V170, V171, V172, V173, V174, V175, V176, V177, V178, V179, V18, V180, V181, V182, V183, V184, V185, V186, V187, V188, V189, V19, V190, V191, V192, V193, V194, V2, V20, V21, V22, V23, V24, V25, V26, V27, V28, V29, V3, V30, V31, V32, V33, V34, V35, V36, V37, V38, V39, V4, V40, V41, V42, V43, V44, V45, V46, V47, V48, V49, V5, V50, V51, V52, V53, V54, V55, V56, V57, V58, V59, V6, V60, V61, V62, V63, V64, V65, V66, V67, V68, V69, V7, V70, V71, V72, V73, V74, V75, V76, V77, V78, V79, V8, V80, V81, V82, V83, V84, V85, V86, V87, V88, V89, V9, V90, V91, V92, V93, V94, V95, V96, V97, V98, V99: VIA, symbol VIA
- added C18, C20, C43, C46, C51, C53, C55: 0u1, symbol C_MINI
- added C42: 120u, symbol C_MINI
- added C44: 1u0, symbol C_MINI
- added C45, C48, C49, C50: 10u, symbol C_MINI
- added C52, C54: 22u, symbol C_MINI
- added D1: MBRX120, symbol D_SCHOTTKY
- added IC10: LM358, symbol OPAMP
- added IC11: 1117-5.0, symbol 1117
- added IC3: TS3USB221DRCR, symbol TS3USB221DRCR
- added IC6: TXB0108, symbol TXB0108_INVERTED
- added IC7: REGULATOR_3.3V, symbol REGULATOR_SOT23-5
- added IC9: AP2101, symbol USB_POWER_SWITCH
- added J1: DC_POWER_JACK, symbol DC_POWER_JACK
- added R40, R41: 15k, symbol R_MINI
- added R42, R43: 10k, symbol R_MINI
- added U1: USB-B, symbol USBCONN
- added U3: microSD, symbol CONN_MICROSD
- added U5: ARDUINO_PINOUT_MICROPENDOUS, symbol ARDUINO_PINOUT_MICROPENDOUS
- added U6: PORTB_3V3, symbol CONN_STK500
- added U7: PORTB, symbol CONN_STK500
- added U8: PORTD, symbol CONN_STK500
- C1, C2: value 24pF -> 24p
- C10: value 1uF -> 1u0
- C11, C35, C36, C39: value 0.1uF -> 0u1
- C12: value 0.01uF -> u01
- C13, C21, C41: value 10uF -> 10u
- C17: value 10uF -> u01
- C37: value 10uF -> 0u1
- F1: value FUSE-MINI -> PolyFuse
- IC1: value AT90USB1287 -> AT90USB1287-AU
- L3: value Ferrite -> FB
- Q1: value MOSFET_P_OPENDOUS -> SI2303
- renumbered L4 to L6
Connections:
- net labels added: PB0_SPI-SS_3.3V, PB1_SPI-SCK_3.3V, PB2_SPI-MOSI_3.3V, PB3_SPI-MISO_3.3V, PB4_3.3V, PB5_3.3V, PB6_3.3V, PB7_3.3V, VBUS_AUX
- net labels removed: EN_OTG, SPI-MISO, SPI-MOSI, SPI-SCK, SPI-SS, USB-A-B-SW, VDD, VT-3.3V-IO0, VT-3.3V-IO1, VT-3.3V-IO2, VT-3.3V-IO3, VT-5V-IO0, VT-5V-IO1, VT-5V-IO2, VT-5V-IO3, VT-EN
- wire segments 281 -> 239
- no-connect marks 6 -> 5
Other:
- note added: "Alternative Part: 74AHC573"
- note added: "Automatically selects"
- note added: "MBR120VLSF"
- note added: "PB0 - SS - PCINT0"
- note added: "PB1 - SCLK - PCINT1"
- note added: "PB2 - MOSI - PCINT2 - PDI"
- note added: "PB3 - MISO - PCINT3 - PDO"
- note added: "PB4 - OC.2A - PCINT4"
- note added: "PB5 - OC.1A - PCINT5"
- note added: "PD0 - OC.0B - SCL - INT0"
- note added: "PD1 - OC.2B - SDA - INT1"
- note added: "PD2 - RXD1 - INT2"
- note added: "PD3 - TXD1 - INT3"
- note added: "PD4 - ICP1"
- note added: "PD5 - XCK1"
- note added: "PD6 - T1"
- note added: "PD7 - T0"
- note added: "PF0 - ADC0"
- note added: "PF1 - ADC1"
- note added: "PF2 - ADC2"
- note added: "PF3 - ADC3"
- note added: "PF4 - ADC4 - JTAG_TCK"
- note added: "PF5 - ADC5 - JTAG_TMS"
- note added: "Power Supply Decoupling"
- note added: "Power Switch for USB-A"
- note added: "SOIC20"
- note added: "SOT223"
- note added: "TS3USB221DRCR has 5V-tolerant control inputs"
- note added: "USB Connector, VIN, or DC Jack"
- note added: "power source between"
- note removed: "DNI"
- note removed: "Do not populate R12, R13"
- note removed: "Optional Footprint"
- note removed: "Populate R1,R2, CR1, CR2, U1 if not"
- note removed: "Populate R2,R3, CR1, CR2, U2 if not"
- note removed: "Populate R5, CR3 to enable OTG"
- note removed: "Use a Logic Level Gate P-Channel MOSFET in DPAK (TO-252)"
- note removed: "need the USB-A connector"
- note removed: "need the USB-B connector"
- note removed: "using the USB switch and you only"
- moved on the sheet: C13, C17, C21, L6, R11, R9, TP1

Commit message: Updated design files for the Micropendous and Micropendous-DIP projects and added pictures for both.  These projects as well as a distribution based on LUFA-101122 are proceeding well.
Parts:
- removed IC3: TS3USB221DRCR, symbol TS3USB221DRCR
- added D2: LED, symbol D_LED
- added IC3: FSUSB20, symbol FSUSB20MUX
- added R42, R45: 1k, symbol R_MINI
- added V101, V103, V104, V11, V111, V114, V12, V121, V124, V125, V128, V136, V14, V149, V15, V153, V154, V155, V156, V157, V16, V160, V168, V174, V175, V183, V185, V187, V188, V189, V19, V190, V195, V196, V197, V198, V204, V207, V219, V22, V222, V223, V224, V225, V226, V23, V231, V232, V235, V236, V237, V238, V239, V24, V240, V241, V242, V243, V246, V248, V252, V253, V254, V255, V256, V257, V258, V259, V26, V260, V261, V262, V263, V264, V265, V266, V267, V268, V269, V27, V270, V271, V272, V273, V274, V276, V277, V278, V279, V28, V280, V281, V282, V283, V284, V285, V286, V287, V288, V289, V29, V290, V291, V292, V293, V294, V295, V296, V297, V298, V299, V3, V30, V300, V301, V302, V303, V304, V305, V306, V307, V308, V309, V310, V311, V312, V313, V314, V315, V316, V317, V318, V319, V320, V321, V322, V323, V324, V325, V326, V327, V328, V329, V330, V331, V332, V333, V334, V336, V339, V34, V340, V341, V342, V343, V344, V345, V346, V347, V348, V349, V35, V350, V351, V352, V36, V37, V38, V39, V40, V42, V45, V46, V51, V52, V53, V54, V55, V56, V57, V59, V6, V60, V61, V62, V63, V64, V65, V66, V68, V82, V83, V86, V87, V90, V99: VIA, symbol VIA
- C42: value 120u -> 47u
- C52: value 22u -> 10u
- IC7: value REGULATOR_3.3V -> REG3V3
- IC9: value AP2101 -> AP2141
- Q1: value SI2303 -> FDN304
- R41: value 15k -> 10k
- renumbered R42 to R44
Connections:
- net labels added: FSUSB_S
- wire segments 239 -> 331
Other:
- note added: "25V+"
- note added: "FSUSB switch also controls USB-A power"
- note added: "FSUSB20 has 7kV of ESD Protection"
- note added: "PB1 = Arduino Pin 13"
- note added: "User LED"
- note removed: "TS3USB221DRCR has 5V-tolerant control inputs"

Commit message: Updated LUFA to LUFA-101122.  Updated LUFAduino, MicropendousKeyboardTest, USBVirtualSerial, and USBVirtualSerial_FreeRTOS firmware demos to LUFA-101122.  Updated Micropendous and Micropendous-DIP hardware designs.
Parts:
- added V353, V354: VIA, symbol VIA
- C42: value 47u -> 100u
- IC5: value CY7C1019D_5V_1MBIT_SRAM -> CY7C1019D-10ZSXI
Connections:
- wire segments 331 -> 337
Other:
- note added: "High Temp."
