File: Micropendous/Design/Micropendous/Micropendous.sch (KiCad schematic (older format))
At the start: 267 parts, among them IC1 AT90USB1287-AU, IC10 LM358, IC11 1117-5.0, IC3 FSUSB20, IC4 74VHC573, IC5 CY7C1019D-10ZSXI, IC6 TXB0108, IC7 REG3V3, IC9 AP2141, J1 DC_POWER_JACK, Q1 FDN304, SW1 RESET, SW2 HWB, U1 USB-B, U2 USB-A, U3 microSD, U4 JTAG, U5 ARDUINO_PINOUT_MICROPENDOUS, U6 PORTB_3V3, U7 PORTB, U8 PORTD, X1 16MHz

Commit message: Partially updated Micropendous design files.  Will add the rest once prototyping is complete.
Parts:
- removed C20: 0u1, symbol C_MINI
- removed C45: 10u, symbol C_MINI
- removed C54: 22u, symbol C_MINI
- removed IC11: 1117-5.0, symbol 1117
- removed IC5: CY7C1019D-10ZSXI, symbol CY7C1019_1MBIT_SRAM
- removed IC7: REG3V3, symbol REGULATOR_SOT23-5
- removed IC9: AP2141, symbol USB_POWER_SWITCH
- removed V267, V270, V301: VIA, symbol VIA
- added C3, C4: 0u1, symbol C_MINI
- added C5: 4u7, symbol C_MINI
- added C54: 22uF, symbol CP_TANTALUM_MINI
- added IC11: MIC39100-5.0WS, symbol REGULATOR_SOT223-3_GND-TAB
- added IC5: IS61C1024AL-12JLI, symbol IS61C1024_IDT71024_1MBIT_SRAM
- added IC7: REG3V3, symbol REGULATOR_SOT89-5_TOREX
- added IC9: AP2140, symbol USB_POWER_SWITCH_ACTIVEHIGH
- added L1: FB, symbol L_MINI
- added Mask1, V1, V10, V100, V13, V17, V18, V2, V20, V21, V25, V31, V32, V33, V4, V41, V43, V44, V47, V48, V49, V5, V50, V58, V67, V69, V7, V70, V71, V72, V73, V74, V75, V76, V77, V78, V79, V8, V80, V81, V84, V85, V88, V89, V9, V91, V92, V93, V94, V95, V96, V97, V98: VIA, symbol VIA
- added R1: DNI, symbol R_MINI
- added U9: Opennect-Controller-MCU_5V-PWR_5W, symbol OPENNECT-CONTROLLER-MCU-PWR
- C17: value u01 -> 10u
- D1: value MBRX120 -> PMEG
- IC4: value 74VHC573 -> 74AHC573
Connections:
- wire segments 337 -> 377
- no-connect marks 5 -> 8
Other:
- note added: "100-Ohm"
- note added: "300-mil SOJ32"
- note added: "Alternative Part: 74VHC573"
- note added: "ESR <2-Ohm"
- note added: "L1 is a copper trace on the board underside that can be\ncut to allow powering PORTB_3V3, the voltage translator,\nand the microSD card from an external 1.2V-3.6V source\nby supplying it to the PORTB_3V3 3V3 pin."
- note added: "MCP1826S-5002E/DB (6V Max Vin)"
- note added: "PMEG3020ER"
- note added: "R1 footprint is included for\ncompatibility with FSUSB30"
- note added: "TSSOP20"
- note added: "Tantalum"
- note added: "XC6210, XC6222, XC6220"
- note removed: "Alternative Part: 74AHC573"
- note removed: "High Temp."
- note removed: "MBR120VLSF"
- note removed: "SOIC20"
- moved on the sheet: C13, C17, C18, C37, C39, C46, C48, C49, C50, C55, IC4, TP2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
