File: Micropendous/Design/Micropendous-DIP/Micropendous-DIP.sch (KiCad schematic (older format))
At the start: 55 parts, among them IC1 AT90USB1287-AU, IC2 AP2101, IC3 TS3USB221, IC4 74VHC573, IC5 CY7C1019D_5V_1MBIT_SRAM, IC6 TXB0108, IC7 REGULATOR_3.3V, P1 Bottom, P2 Top, P3 PB_3.3V, SW1 RESET, SW2 HWB, U1 USB-miniB, U2 USB-A, U3 CONN_MICROSD, U4 JTAG, X1 16MHz

Commit message: Updated Micropendous and Micropendous-DIP AT90USB1287-based designs.
Parts:
- removed CR1, CR2: ESD_ZENER, symbol ESD_ZENER
- removed IC2: AP2101, symbol USB_SWITCH
- removed IC3: TS3USB221, symbol TS3USB221
- removed R1, R2: 0, symbol R_MINI
- added C49, C50: 10u, symbol C_MINI
- added IC2: AP2101, symbol USB_POWER_SWITCH
- added IC3: FSUSB20, symbol FSUSB20MUX
- added R41: 15k, symbol R_MINI
- added V101, V102, V103, V104, V11, V111, V114, V12, V121, V124, V125, V128, V133, V135, V136, V14, V149, V15, V150, V151, V153, V154, V155, V156, V157, V16, V160, V161, V162, V168, V171, V172, V173, V174, V175, V183, V185, V187, V188, V189, V19, V190, V195, V196, V197, V198, V199, V200, V201, V202, V203, V204, V205, V207, V209, V210, V211, V212, V213, V214, V215, V216, V217, V218, V219, V22, V220, V222, V223, V224, V225, V226, V227, V228, V229, V23, V230, V231, V232, V233, V235, V236, V237, V238, V239, V24, V240, V241, V242, V243, V246, V248, V252, V253, V254, V255, V256, V257, V258, V259, V26, V260, V261, V262, V263, V264, V265, V266, V27, V28, V29, V3, V30, V34, V35, V36, V37, V38, V39, V40, V42, V45, V46, V47, V51, V52, V53, V54, V55, V56, V57, V59, V6, V60, V61, V62, V63, V64, V65, V66, V68, V82, V83, V86, V87, V90, V91, V92, V99: VIA, symbol VIA
- C10, C44: value 1uF -> 1u0
- C11, C18, C20, C35, C36, C37, C39, C43, C46: value 0.1uF -> 0u1
- C12, C17: value 0.01uF -> u01
- C13, C21, C41, C45, C48: value 10uF -> 10u
- C42: value 120uF -> 120u
- L3: value Ferrite -> FB
- R40, R9: value 10k -> 15k
- U3: value CONN_MICROSD -> microSD
Connections:
- net labels removed: VT-EN
- wire segments 176 -> 245
- no-connect marks 4 -> 5
Other:
- note added: "Depopulate L5 to enable powering the board"
- note added: "TQFP Package has no GND-PAD"
- note added: "through the VDD5 pin on the top header"
- note removed: "Only the USB-miniB connector U1 will function"
- note removed: "Populate R1, R2, CR1, CR2, U1 if not"
- note removed: "using the USB switch (IC3, U2)"
- moved on the sheet: C13, C18, C20, C21, C37, C42, C43, C44, C45, C46, L5, R11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

Commit message: Updated Micropendous-DIP with series resistor from PE7 to FSUSB20 control pin to act as a simple voltage translator.
Parts:
- added R42: 1k, symbol R_MINI
- added V267: VIA, symbol VIA
- L5: value Ferrite -> FB
- R41: value 15k -> 10k
Connections:
- net labels added: FSUSB_S
Changed lines of the file:
@@
-EESchema Schematic File Version 2  date 10/10/2010 02:01:42
+EESchema Schematic File Version 2  date 14/10/2010 04:24:29
 LIBS:power
 LIBS:device
@@
 LIBS:valves
 LIBS:opendous
-LIBS:Micropendous-DIP-cache
 EELAYER 24  0
 EELAYER END
@@
 Sheet 1 1
 Title "Micropendous-DIP"
-Date "4 oct 2010"
+Date "14 oct 2010"
 Rev "1.1"
 Comp ""
@@
 Comment4 "www.Micropendous.org"
 $EndDescr
+Text Label 7600 7950 0    20   ~ 0
+FSUSB_S
 $Comp
-L VIA V266
-U 1 1 4CA99C6F
-P 7200 8250
-F 0 "V266" V 7225 8350 20  0000 C CNN
-F 1 "VIA" H 7200 8450 60  0001 C CNN
-	1    7200 8250
+L VIA V267
+U 1 1 4CB6BA0D
+P 7600 7950
+F 0 "V267" V 7625 8050 20  0000 C CNN
+F 1 "VIA" H 7600 8150 60  0001 C CNN
+	1    7600 7950
 	0    -1   -1   0
 $EndComp
 Text Label 7200 8250 0    20   ~ 0
-PE7
-$Comp
-L VDD33 #PWR01
-U 1 1 4CA99C1E
-P 7250 8200
-F 0 "#PWR01" H 7250 8300 30  0001 C CNN
-F 1 "VDD33" V 7250 8350 30  0000 C CNN
-	1    7250 8200
-	0    1    1    0
-$EndComp
-$Comp
-L VIA V265
-U 1 1 4CA99C11
-P 7200 8200
-F 0 "V265" V 7225 8300 20  0000 C CNN
-F 1 "VIA" H 7200 8400 60  0001 C CNN
-	1    7200 8200
-	0    -1   -1   0
-$EndComp
+FSUSB_S
+Text Label 3300 1900 0    20   ~ 0
+FSUSB_S
+Connection ~ 3500 1900
+Wire Wire Line
+	3300 1900 3700 1900
+Wire Wire Line
+	3500 1900 3500 1650
 Wire Wire Line
 	7200 8200 7250 8200
@@
 Wire Wire Line
 	550  8225 550  7925
-Wire Wire Line
-	3500 1650 3500 1900
-Wire Wire Line
-	3500 1900 3300 1900
 Connection ~ 7200 8000
 Connection ~ 7200 7950
@@
 	3300 1350 3300 1450
 $Comp
+L R_MINI R42
+U 1 1 4CB6B751
+P 3800 1900
+F 0 "R42" H 3730 1950 25  0000 C CNN
+F 1 "1k" H 3870 1950 20  0000 C CNN
+	1    3800 1900
+	1    0    0    -1
+$EndComp
+$Comp
+L VIA V266
+U 1 1 4CA99C6F
+P 7200 8250
+F 0 "V266" V 7225 8350 20  0000 C CNN
+F 1 "VIA" H 7200 8450 60  0001 C CNN
+	1    7200 8250
+	0    -1   -1   0
+$EndComp
+$Comp
+L VDD33 #PWR01
+U 1 1 4CA99C1E
+P 7250 8200
+F 0 "#PWR01" H 7250 8300 30  0001 C CNN
+F 1 "VDD33" V 7250 8350 30  0000 C CNN
+	1    7250 8200
+	0    1    1    0
+$EndComp
+$Comp
+L VIA V265
+U 1 1 4CA99C11
+P 7200 8200
+F 0 "V265" V 7225 8300 20  0000 C CNN
+F 1 "VIA" H 7200 8400 60  0001 C CNN
+	1    7200 8200
+	0    -1   -1   0
+$EndComp
+$Comp
 L FSUSB20MUX IC3
 U 1 1 4CA995A7
@@
 P 3500 1550
 F 0 "R41" V 3475 1600 25  0000 C CNN
-F 1 "15k" V 3525 1600 20  0000 C CNN
+F 1 "10k" V 3525 1600 20  0000 C CNN
 	1    3500 1550
 	0    1    1    0
@@
 P 9750 3500
 F 0 "L5" H 9675 3450 30  0000 C CNN
-F 1 "Ferrite" H 9800 3450 22  0000 C CNN
+F 1 "FB" H 9800 3450 22  0000 C CNN
 	1    9750 3500
 	-1   0    0    1
@@
 	1    0    0    -1
 $EndComp
-Text Label 3300 1900 0    20   ~ 0
+Text Label 3900 1900 0    20   ~ 0
 PE7
 Text Label 1800 2200 0    20   ~ 0

Commit message: Updated LUFA to LUFA-101122.  Updated LUFAduino, MicropendousKeyboardTest, USBVirtualSerial, and USBVirtualSerial_FreeRTOS firmware demos to LUFA-101122.  Updated Micropendous and Micropendous-DIP hardware designs.
Parts:
- removed L5: FB, symbol L_MINI
- added F1: PTC, symbol FUSE-MINI
Connections:
- wire segments 245 -> 252
Other:
- note added: "Depopulate F1 to enable powering the board"
- note added: "This may also be a jumper"
- note removed: "Depopulate L5 to enable powering the board"
