File: Micropendous/Design/Micropendous-Eth/Micropendous-Eth.sch (KiCad schematic (older format))
At the start: 267 parts, among them IC1 AT90USB1287-AU, IC10 LM358, IC11 1117-5.0, IC3 FSUSB20, IC4 74VHC573, IC5 CY7C1019D-10ZSXI, IC6 TXB0108, IC7 REG3V3, IC9 AP2141, J1 DC_POWER_JACK, Q1 FDN304, SW1 RESET, SW2 HWB, U1 USB-B, U2 USB-A, U3 microSD, U4 JTAG, U5 ARDUINO_PINOUT_MICROPENDOUS, U6 PORTB_3V3, U7 PORTB, U8 PORTD, X1 16MHz

Commit message: Added Micropendous-32U2 and Micropendous-ETH designs.  Minor updates to other hardware designs.
Parts:
- removed C51, C53: 0u1, symbol C_MINI
- removed C52: 10u, symbol C_MINI
- removed C54: 22u, symbol C_MINI
- removed D1: MBRX120, symbol D_SCHOTTKY
- removed IC10: LM358, symbol OPAMP
- removed IC11: 1117-5.0, symbol 1117
- removed J1: DC_POWER_JACK, symbol DC_POWER_JACK
- removed Q1: FDN304, symbol MOSFET_P_OPENDOUS
- removed R43, R44: 10k, symbol R_MINI
- removed V42, V53, V56: VIA, symbol VIA
- added C56, C57: 24p, symbol C_MINI
- added C58: 10u, symbol C_MINI
- added C59, C60, C61, C62, C63, C64, C65: 0u1, symbol C_MINI
- added IC10: ENC28J60, symbol ENC28J60_QFN
- added J1: PULSE_J00-00__NL, symbol PULSE_J00-00_PHY_SIDE
- added L7: FB, symbol L_MINI
- added R47: 2k32, symbol R_MINI
- added R48, R49, R50, R51: 49.9, symbol R_MINI
- added R52, R53: 100, symbol R_MINI
- added V355, V356, V357, V358, V359, V360, V361, V362: VIA, symbol VIA
- added X2: 25MHz, symbol CRYSTAL
- F1: value PolyFuse -> PTC
Connections:
- net labels added: CT_TD, FS_nOE, LEDA, LEDB, RBIAS, RD+, RD-, TD+, TD-, VCAP
- wire segments 337 -> 363
- no-connect marks 5 -> 9
Other:
- note added: "1%"
- note added: "Low ESR X?R"
- note added: "PolyFuse"
- note added: "VIN Not Connected"
- note removed: "25V+"
- note removed: "Automatically selects"
- note removed: "High Temp."
- note removed: "MBR120VLSF"
- note removed: "SOT223"
- note removed: "USB Connector, VIN, or DC Jack"
- note removed: "power source between"
- moved on the sheet: F1, IC3, L6, R11, R41, R42, R9, TP1, U1, U2, U4
