File: Micropendous/Design/Micropendous-OTG/Micropendous.sch (KiCad schematic (older format))
At the start: 322 parts, among them IC1 AT90USB1287-AU, IC10 LM358, IC11 MIC39100-5.0WS, IC3 FSUSB30, IC4 74AHC573, IC5 IS61C1024AL-12JLI, IC6 TXB0108, IC7 REG3V3, IC9 AP2151, J1 DC_POWER_JACK, Q1 FDN304, SW1 RESET, SW2 HWB, U1 USB-B, U2 USB-A, U3 microSD, U4 JTAG, U5 ARDUINO_PINOUT_MICROPENDOUS, U6 PORTB_3V3, U7 PORTB, U8 PORTD, U9 Opennect-Controller-MCU_5V-PW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, X1 16MHz

Commit message: Added new version of Micropendous (Arduino-like) design.  Moved the old version to Micropendous-OTG.  Micropendous-OTG was based on the Micropendous-DIP schematic which includes OTG capability.  The new Micropendous version focuses on Device and Host modes and the OTG pin (PE3) is used to control the voltage translator.
Parts:
- removed L2: FB, symbol L_MINI
- removed V102: VIA, symbol VIA
- added L6: FB, symbol L_MINI
- C1, C2: value 18p -> 24p
- C43: value u01 -> 0u1
- C5: value 1u0 -> 4u7
- IC3: value FSUSB30 -> FSUSB20
- IC9: value AP2151 -> AP2140
- R1: value 100 -> DNI
- R11, R40, R9: value 10k -> 15k
- R42: value 5k1 -> 1k
Connections:
- wire segments 369 -> 377
- no-connect marks 9 -> 8
Other:
- note added: "100-Ohm"
- note added: "ESR <2-Ohm"
- note added: "FSUSB switch also controls USB-A power"
- note added: "FSUSB20 has 7kV of ESD Protection"
- note added: "R1 footprint is included for\ncompatibility with FSUSB30"
- note added: "XC6210, XC6222, XC6220"
- note removed: "0.2-Ohm < ESR <1-Ohm"
- note removed: "50ppm or better frequency\nstability is required by USB"
- note removed: "FSUSB switch also\ncontrols USB-A power"
- note removed: "FSUSB30 has 8kV of ESD Protection"
- note removed: "Intel USB Design Guidelines\nrecommend Low ESR (<100mOhm)\ncapacitors of 120uF+ to allow for\ntemperature derating. Ceramic\n100uF is the simplest solution."
- note removed: "Only Compatible with Opennect-MCU\nstandard if using CUI EMSA060300-P5P-SZ\nor Volgen KTPS24-06035MP wall adapter\npower supply outputting about 3A at 6V\n850mA rating takes into account trace width"
- note removed: "R1 should be anti-surge or\npulse-withstanding"
- note removed: "XC6220B331PR-G"
- note removed: "XC6222B331PR-G"
- moved on the sheet: C13, C17, C18, C21, C3, C37, C39, C4, C42, C43, C44, C46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
